Commit message: [ADD] agibot A2D and fftai gr1t1

File: urdf/A2D.urdf (robot description, URDF)
Before this commit: robot A2D, 42 links, 41 joints
Links:
- link Link1_l: geometry collision mesh filename=meshes/A2D/Link1_l.STL; visual mesh filename=meshes/A2D/Link1_l.STL
- link Link1_r: geometry collision mesh filename=meshes/A2D/Link1_r.STL; visual mesh filename=meshes/A2D/Link1_r.STL
- link Link2_l: geometry collision mesh filename=meshes/A2D/Link2_l.STL; visual mesh filename=meshes/A2D/Link2_l.STL
- link Link2_r: geometry collision mesh filename=meshes/A2D/Link2_r.STL; visual mesh filename=meshes/A2D/Link2_r.STL
- link Link3_l: geometry collision mesh filename=meshes/A2D/Link3_l.STL; visual mesh filename=meshes/A2D/Link3_l.STL
- link Link3_r: geometry collision mesh filename=meshes/A2D/Link3_r.STL; visual mesh filename=meshes/A2D/Link3_r.STL
- link Link4_l: geometry collision mesh filename=meshes/A2D/Link4_l.STL; visual mesh filename=meshes/A2D/Link4_l.STL
- link Link4_r: geometry collision mesh filename=meshes/A2D/Link4_r.STL; visual mesh filename=meshes/A2D/Link4_r.STL
- link Link5_l: geometry collision mesh filename=meshes/A2D/Link5_l.STL; visual mesh filename=meshes/A2D/Link5_l.STL
- link Link5_r: geometry collision mesh filename=meshes/A2D/Link5_r.STL; visual mesh filename=meshes/A2D/Link5_r.STL
- link Link6_l: geometry collision mesh filename=meshes/A2D/Link6_l.STL; visual mesh filename=meshes/A2D/Link6_l.STL
- link Link6_r: geometry collision mesh filename=meshes/A2D/Link6_r.STL; visual mesh filename=meshes/A2D/Link6_r.STL
- link Link7_l: geometry collision mesh filename=meshes/A2D/Link7_l.STL; visual mesh filename=meshes/A2D/Link7_l.STL
- link Link7_r: geometry collision mesh filename=meshes/A2D/Link7_r.STL; visual mesh filename=meshes/A2D/Link7_r.STL
- link base_link: geometry collision mesh filename=meshes/A2D/base_link.STL; visual mesh filename=meshes/A2D/base_link.STL
- link base_link_l: geometry collision mesh filename=meshes/A2D/base_link_l.STL; visual mesh filename=meshes/A2D/base_link_l.STL
- link base_link_r: geometry collision mesh filename=meshes/A2D/base_link_r.STL; visual mesh filename=meshes/A2D/base_link_r.STL
- link left_base_link: geometry collision mesh filename=meshes/A2D/gripper_base_link.STL; visual mesh filename=meshes/A2D/gripper_base_link.STL
- link left_narrow1_Link: geometry collision mesh filename=meshes/A2D/narrow1_Link.STL; visual mesh filename=meshes/A2D/narrow1_Link.STL
- link left_narrow2_Link: geometry collision mesh filename=meshes/A2D/narrow2_Link.STL; visual mesh filename=meshes/A2D/narrow2_Link.STL
- link left_narrow3_Link: geometry collision mesh filename=meshes/A2D/narrow3_Link.STL; visual mesh filename=meshes/A2D/narrow3_Link.STL
- link left_narrow4_Link: geometry collision mesh filename=meshes/A2D/narrow4_Link.STL; visual mesh filename=meshes/A2D/narrow4_Link.STL
- link left_wide1_Link: geometry collision mesh filename=meshes/A2D/wide1_Link.STL; visual mesh filename=meshes/A2D/wide1_Link.STL
- link left_wide2_Link: geometry collision mesh filename=meshes/A2D/wide2_Link.STL; visual mesh filename=meshes/A2D/wide2_Link.STL
- link left_wide3_Link: geometry collision mesh filename=meshes/A2D/wide3_Link.STL; visual mesh filename=meshes/A2D/wide3_Link.STL
- link left_wide4_Link: geometry collision mesh filename=meshes/A2D/wide4_Link.STL; visual mesh filename=meshes/A2D/wide4_Link.STL
- link link_pitch_body: geometry collision mesh filename=meshes/A2D/link_pitch_body.STL; visual mesh filename=meshes/A2D/link_pitch_body.STL
- link link_pitch_head: geometry collision mesh filename=meshes/A2D/link_pitch_head.STL; visual mesh filename=meshes/A2D/link_pitch_head.STL
- link link_up_down_body: geometry collision mesh filename=meshes/A2D/link_up_down_body.STL; visual mesh filename=meshes/A2D/link_up_down_body.STL
- link link_yaw_head: geometry collision mesh filename=meshes/A2D/link_yaw_head.STL; visual mesh filename=meshes/A2D/link_yaw_head.STL
- link right_base_link: geometry collision mesh filename=meshes/A2D/gripper_base_link.STL; visual mesh filename=meshes/A2D/gripper_base_link.STL
- link right_narrow1_Link: geometry collision mesh filename=meshes/A2D/narrow1_Link.STL; visual mesh filename=meshes/A2D/narrow1_Link.STL
- link right_narrow2_Link: geometry collision mesh filename=meshes/A2D/narrow2_Link.STL; visual mesh filename=meshes/A2D/narrow2_Link.STL
- link right_narrow3_Link: geometry collision mesh filename=meshes/A2D/narrow3_Link.STL; visual mesh filename=meshes/A2D/narrow3_Link.STL
- link right_narrow4_Link: geometry collision mesh filename=meshes/A2D/narrow4_Link.STL; visual mesh filename=meshes/A2D/narrow4_Link.STL
- link right_wide1_Link: geometry collision mesh filename=meshes/A2D/wide1_Link.STL; visual mesh filename=meshes/A2D/wide1_Link.STL
- link right_wide2_Link: geometry collision mesh filename=meshes/A2D/wide2_Link.STL; visual mesh filename=meshes/A2D/wide2_Link.STL
- link right_wide3_Link: geometry collision mesh filename=meshes/A2D/wide3_Link.STL; visual mesh filename=meshes/A2D/wide3_Link.STL
- link right_wide4_Link: geometry collision mesh filename=meshes/A2D/wide4_Link.STL; visual mesh filename=meshes/A2D/wide4_Link.STL
