Commit message: [Add] r1 lite dae files

File: urdf/r1_lite.urdf (robot description, URDF)
Before this commit: robot mmp_revB_invconfig_upright_a1x, 34 links, 33 joints
Links:
- link base_link: geometry collision mesh filename=meshes/r1_lite/base_link_collision.STL; visual mesh filename=meshes/r1_lite/base_link.dae
- link left_D405_link: geometry collision mesh filename=meshes/r1_lite/left_D405_link_collision.STL; visual mesh filename=meshes/r1_lite/left_D405_link.dae
- link left_arm_base_link: geometry collision mesh filename=meshes/r1_lite/left_arm_base_link_collision.STL; visual mesh filename=meshes/r1_lite/left_arm_base_link.dae
- link left_arm_link1: geometry collision mesh filename=meshes/r1_lite/left_arm_link1_collision.STL; visual mesh filename=meshes/r1_lite/left_arm_link1.dae
- link left_arm_link2: geometry collision mesh filename=meshes/r1_lite/left_arm_link2_collision.STL; visual mesh filename=meshes/r1_lite/left_arm_link2.dae
- link left_arm_link3: geometry collision mesh filename=meshes/r1_lite/left_arm_link3_collision.STL; visual mesh filename=meshes/r1_lite/left_arm_link3.dae
- link left_arm_link4: geometry collision mesh filename=meshes/r1_lite/left_arm_link4_collision.STL; visual mesh filename=meshes/r1_lite/left_arm_link4.dae
- link left_arm_link5: geometry collision mesh filename=meshes/r1_lite/left_arm_link5_collision.STL; visual mesh filename=meshes/r1_lite/left_arm_link5.dae
- link left_arm_link6: geometry collision mesh filename=meshes/r1_lite/left_arm_link6_collision.STL; visual mesh filename=meshes/r1_lite/left_arm_link6.dae
- link left_gripper_finger_link1: geometry collision box size=0.06 0.01 0.04; visual mesh filename=meshes/r1_lite/left_gripper_finger_link1.dae
- link left_gripper_finger_link2: geometry collision box size=0.06 0.01 0.04; visual mesh filename=meshes/r1_lite/left_gripper_finger_link2.dae
- link left_gripper_link: geometry collision mesh filename=meshes/r1_lite/left_gripper_link_collision.STL; visual mesh filename=meshes/r1_lite/left_gripper_link.dae
- link right_D405_link: geometry collision mesh filename=meshes/r1_lite/right_D405_link_collision.STL; visual mesh filename=meshes/r1_lite/right_D405_link.dae
- link right_arm_base_link: geometry collision mesh filename=meshes/r1_lite/right_arm_base_link_collision.STL; visual mesh filename=meshes/r1_lite/right_arm_base_link.dae
- link right_arm_link1: geometry collision mesh filename=meshes/r1_lite/right_arm_link1_collision.STL; visual mesh filename=meshes/r1_lite/right_arm_link1.dae
- link right_arm_link2: geometry collision mesh filename=meshes/r1_lite/right_arm_link2_collision.STL; visual mesh filename=meshes/r1_lite/right_arm_link2.dae
- link right_arm_link3: geometry collision mesh filename=meshes/r1_lite/right_arm_link3_collision.STL; visual mesh filename=meshes/r1_lite/right_arm_link3.dae
- link right_arm_link4: geometry collision mesh filename=meshes/r1_lite/right_arm_link4_collision.STL; visual mesh filename=meshes/r1_lite/right_arm_link4.dae
- link right_arm_link5: geometry collision mesh filename=meshes/r1_lite/right_arm_link5_collision.STL; visual mesh filename=meshes/r1_lite/right_arm_link5.dae
- link right_arm_link6: geometry collision mesh filename=meshes/r1_lite/right_arm_link6_collision.STL; visual mesh filename=meshes/r1_lite/right_arm_link6.dae
- link right_gripper_finger_link1: geometry collision box size=0.06 0.01 0.04; visual mesh filename=meshes/r1_lite/right_gripper_finger_link1.dae
- link right_gripper_finger_link2: geometry collision box size=0.06 0.01 0.04; visual mesh filename=meshes/r1_lite/right_gripper_finger_link2.dae
- link right_gripper_link: geometry collision mesh filename=meshes/r1_lite/right_gripper_link_collision.STL; visual mesh filename=meshes/r1_lite/right_gripper_link.dae
- link steer_motor_link1: geometry collision mesh filename=meshes/r1_lite/steer_motor_link1_collision.STL; visual mesh filename=meshes/r1_lite/steer_motor_link1.dae
- link steer_motor_link2: geometry collision mesh filename=meshes/r1_lite/steer_motor_link2_collision.STL; visual mesh filename=meshes/r1_lite/steer_motor_link2.dae
- link steer_motor_link3: geometry collision mesh filename=meshes/r1_lite/steer_motor_link3_collision.STL; visual mesh filename=meshes/r1_lite/steer_motor_link3.dae
- link torso_link1: geometry collision mesh filename=meshes/r1_lite/torso_link1_collision.STL; visual mesh filename=meshes/r1_lite/torso_link1.dae
- link torso_link2: geometry collision mesh filename=meshes/r1_lite/torso_link2_collision.STL; visual mesh filename=meshes/r1_lite/torso_link2.dae
- link torso_link3: geometry collision mesh filename=meshes/r1_lite/torso_link3_collision.STL; visual mesh filename=meshes/r1_lite/torso_link3.dae
- link wheel_motor_link1: geometry collision mesh filename=meshes/r1_lite/wheel_motor_link1_collision.STL; visual mesh filename=meshes/r1_lite/wheel_motor_link1.dae
- link wheel_motor_link2: geometry collision mesh filename=meshes/r1_lite/wheel_motor_link2_collision.STL; visual mesh filename=meshes/r1_lite/wheel_motor_link2.dae
- link wheel_motor_link3: geometry collision mesh filename=meshes/r1_lite/wheel_motor_link3_collision.STL; visual mesh filename=meshes/r1_lite/wheel_motor_link3.dae
