Commit message: [Fix] urdf gripper file name

File: urdf/grippers.urdf (robot description, URDF)
Before this commit: robot DAS Final-818-819-URDF, 3 links, 2 joints
Links:
- link left_hand: geometry collision mesh filename=./gripper_hand.glb; visual mesh filename=./gripper_hand.glb scale=0.1 0.1 0.1
- link right_hand: geometry collision mesh filename=./gripper_hand.glb; visual mesh filename=./gripper_hand.glb scale=0.1 0.1 0.1
